File: HP45 Standalone V4.02.kicad_pcb (KiCad board)
At the start: 2 copper layers, 44 x 100 mm, 90 parts, among them Con1 HP45_connector, IC1 ADP2301, IC2 74HC123, IC3 TLC59213, IC4 TLC59213, IC5 HEF4017, IC6 HEF4017, IC7 HCF4081, IC8 LM311, IC9 HEF4017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

Commit message: Power input
Other:
- net class Default removed
- net class Power removed
