File: HP45 Standalone V4.02.kicad_sch (KiCad schematic)
At the start: 25 parts, among them IC2 LM311, M1 Mounting_hole, M2 Mounting_hole, M3 Mounting_hole, M4 Mounting_hole, Q1 Q_NMOS_SGD

Commit message: complete schema
Other:
- added sheet HP45 (HP45.kicad_sch)
Changed lines of the file:
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@@
+    )
+  )
+  (sheet (at 21.59 126.365) (size 13.97 3.81) (fields_autoplaced)
+    (stroke (width 0.1524) (type solid))
+    (fill (color 0 0 0 0.0000))
+    (property "Sheetname" "HP45" (at 21.59 125.6534 0)
+      (effects (font (size 1.27 1.27)) (justify left bottom))
+    )
+    (property "Sheetfile" "HP45.kicad_sch" (at 21.59 130.7596 0)
+      (effects (font (size 1.27 1.27)) (justify left top))
+    )
+    (instances
+      (project "HP45 Standalone V4.02"
+        (path "/1b59a1f1-c87a-43e4-bb42-f8c258f5ff1e" (page "3"))
+      )
     )
   )
